Commit message: Refactoring

File: assets/robots/ur10e.urdf (robot description, URDF)
Before this commit: robot ur10e, 26 links, 25 joints
Links:
- removed link tcp_link
- added link robotiq140_tcp_link, mass 0.0
Joints:
- removed joint tcp_joint
- added joint robotiq140_tcp_joint: type fixed, parent realsense_mount_base_link, child robotiq140_tcp_link, origin xyz=0 0 0.22 rpy=0 0 0
